File: attiny84-l298/attiny84-l298.kicad_pcb (KiCad board)
At the start: 2 copper layers, 160 x 100 mm, 29 parts, among them J1 DIN41612_02x16_AB, J2 Banana Socket, J3 Banana Socket, J4 Banana Socket, J5 Banana Socket, SW1 SW_DIP_x08, U1 74151, U2 ATtiny84A-P, U3 L298HN

Commit message: Cleaned up schematic and fixed DRC errors
Signed-off-by: Matthew Nickson <mnickson@sidingsmedia.com>
Connections:
- J1 pad a1: +12V -> unconnected-(J1-Pada1)
- J1 pad a10: /SPI_SCLK -> unconnected-(J1-Pada10)
- J1 pad a11: /SPI_MOSI -> unconnected-(J1-Pada11)
- J1 pad a12: /SPI_MISO -> unconnected-(J1-Pada12)
- J1 pad a13: /SPI_~{CS_{1}} -> unconnected-(J1-Pada13)
- J1 pad a14: /SPI_~{CS_{2}} -> unconnected-(J1-Pada14)
- J1 pad a2: +12V -> unconnected-(J1-Pada2)
- J1 pad a3: -12V -> unconnected-(J1-Pada3)
- J1 pad a4: -12V -> unconnected-(J1-Pada4)
- J1 pad a5: +3V3 -> unconnected-(J1-Pada5)
- J1 pad a6: +3V3 -> unconnected-(J1-Pada6)
- J1 pad b11: /UD/NC -> unconnected-(J1-Padb11)
- J1 pad b12: /UD/NC -> unconnected-(J1-Padb12)
- J1 pad b13: /UD/NC -> unconnected-(J1-Padb13)
- J1 pad b14: /UD/NC -> unconnected-(J1-Padb14)
- J1 pad b15: /SPI_~{CS_{4}} -> unconnected-(J1-Padb15)
- J1 pad b16: /SPI_~{CS_{3}} -> unconnected-(J1-Padb16)
- J1 pad b3: -5V -> unconnected-(J1-Padb3)
- J1 pad b4: -5V -> unconnected-(J1-Padb4)
- J1 pad b5: +1V1 -> unconnected-(J1-Padb5)
- J1 pad b6: +1V1 -> unconnected-(J1-Padb6)
- J3 pad 2: (no net) -> GND
- J3 pad 3: (no net) -> GND
