File: attiny84/attiny84.kicad_sch (KiCad schematic)
At the start: 30 parts, among them J1 DIN41612_02x16_AB, J2 USB_C_Receptacle_USB2.0, Q1 BSS138, Q2 BSS138, Q4 DMG2305UX, SW2 SW_Push, U1 MCP2221AxSL, U2 ATtiny84A-P

Commit message: Assigned footprints to all components
Signed-off-by: Matthew Nickson <mnickson@sidingsmedia.com>
Parts:
- C1, C4: footprint (none) -> Capacitor_SMD:C_1206_3216Metric_Pad1.33x1.80mm_HandSolder
- C2, C3: footprint Capacitor_THT:C_Disc_D4.7mm_W2.5mm_P5.00mm -> Capacitor_SMD:C_1206_3216Metric_Pad1.33x1.80mm_HandSolder
- D1, D2, D3, D4: footprint (none) -> Capacitor_SMD:C_0402_1005Metric_Pad0.74x0.62mm_HandSolder
- H1, H2, H3, H4: footprint (none) -> MountingHole:MountingHole_2.7mm
- J2: footprint (none) -> Connector_USB:USB_C_Receptacle_Palconn_UTC16-G
- R1, R16, R2, R3: footprint (none) -> Resistor_SMD:R_1206_3216Metric_Pad1.30x1.75mm_HandSolder
- R10: footprint Resistor_THT:R_Axial_DIN0207_L6.3mm_D2.5mm_P7.62mm_Horizontal -> Resistor_SMD:R_1206_3216Metric_Pad1.30x1.75mm_HandSolder
- R12, R13, R14, R15: footprint Resistor_SMD:R_0805_2012Metric -> Resistor_SMD:R_1206_3216Metric_Pad1.30x1.75mm_HandSolder
- U2: footprint Package_DIP:DIP-14_W7.62mm -> Package_SO:SOIC-14_3.9x8.7mm_P1.27mm

Commit message: Changed hole refference to match other schematics
Signed-off-by: Matthew Nickson <mnickson@sidingsmedia.com>
Parts:
- renumbered H1 to MK1, H2 to MK2, H3 to MK3, H4 to MK4
Changed lines of the file:
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@@
   (symbol (lib_id "Mechanical:MountingHole_Pad") (at 15.24 193.04 0) (unit 1)
     (in_bom yes) (on_board yes) (fields_autoplaced)
-    (property "Reference" "H4" (id 0) (at 17.78 190.4999 0)
+    (property "Reference" "MK4" (id 0) (at 17.78 190.4999 0)
       (effects (font (size 1.27 1.27)) (justify left))
     )
@@
   (symbol (lib_id "Mechanical:MountingHole_Pad") (at 15.24 185.42 0) (unit 1)
     (in_bom yes) (on_board yes) (fields_autoplaced)
-    (property "Reference" "H3" (id 0) (at 17.78 182.8799 0)
+    (property "Reference" "MK3" (id 0) (at 17.78 182.8799 0)
       (effects (font (size 1.27 1.27)) (justify left))
     )
@@
   (symbol (lib_id "Mechanical:MountingHole_Pad") (at 15.24 170.18 0) (unit 1)
     (in_bom yes) (on_board yes) (fields_autoplaced)
-    (property "Reference" "H1" (id 0) (at 17.78 167.6399 0)
+    (property "Reference" "MK1" (id 0) (at 17.78 167.6399 0)
       (effects (font (size 1.27 1.27)) (justify left))
     )
@@
   (symbol (lib_id "Mechanical:MountingHole_Pad") (at 15.24 177.8 0) (unit 1)
     (in_bom yes) (on_board yes) (fields_autoplaced)
-    (property "Reference" "H2" (id 0) (at 17.78 175.2599 0)
+    (property "Reference" "MK2" (id 0) (at 17.78 175.2599 0)
       (effects (font (size 1.27 1.27)) (justify left))
     )
@@
       (reference "F1") (unit 1) (value "5A") (footprint "Fuse:Fuseholder_Littelfuse_445_030_series_5x20mm")
     )
-    (path "/8ae9a3f2-0a72-43b1-a632-5c7588c9710d"
-      (reference "H1") (unit 1) (value "MountingHole_Pad") (footprint "MountingHole:MountingHole_2.7mm")
-    )
-    (path "/caf60ef0-6398-47f8-83aa-2549673c7f6c"
-      (reference "H2") (unit 1) (value "MountingHole_Pad") (footprint "MountingHole:MountingHole_2.7mm")
-    )
-    (path "/70ecdcb3-2b1d-4dbb-9c29-b8eb242f418b"
-      (reference "H3") (unit 1) (value "MountingHole_Pad") (footprint "MountingHole:MountingHole_2.7mm")
-    )
-    (path "/06e3cd8a-7f61-4bd0-a023-8cd89c2cd84e"
-      (reference "H4") (unit 1) (value "MountingHole_Pad") (footprint "MountingHole:MountingHole_2.7mm")
-    )
     (path "/dad53da1-1ed9-4f5a-866b-6bc10822e80b"
       (reference "J1") (unit 1) (value "DIN41612_02x16_AB") (footprint "Connector_DIN:DIN41612_B2_2x16_Male_Horizontal_THT")
@@
       (reference "J6") (unit 1) (value "Screw_Terminal_01x03") (footprint "TerminalBlock:TerminalBlock_bornier-3_P5.08mm")
     )
+    (path "/8ae9a3f2-0a72-43b1-a632-5c7588c9710d"
+      (reference "MK1") (unit 1) (value "MountingHole_Pad") (footprint "MountingHole:MountingHole_2.7mm")
+    )
+    (path "/caf60ef0-6398-47f8-83aa-2549673c7f6c"
+      (reference "MK2") (unit 1) (value "MountingHole_Pad") (footprint "MountingHole:MountingHole_2.7mm")
+    )
+    (path "/70ecdcb3-2b1d-4dbb-9c29-b8eb242f418b"
+      (reference "MK3") (unit 1) (value "MountingHole_Pad") (footprint "MountingHole:MountingHole_2.7mm")
+    )
+    (path "/06e3cd8a-7f61-4bd0-a023-8cd89c2cd84e"
+      (reference "MK4") (unit 1) (value "MountingHole_Pad") (footprint "MountingHole:MountingHole_2.7mm")
+    )
     (path "/5f363ae9-a03f-479d-856e-b8161074866b"

Commit message: Removed left over net label from IN1
Signed-off-by: Matthew Nickson <mnickson@sidingsmedia.com>
Connections:
- net IN1 renamed Motor Driver/IN1
Changed lines of the file:
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@@
     (effects (font (size 1.27 1.27)) (justify left bottom))
-  )
-  (label "IN1" (at 149.86 73.66 180)
-    (effects (font (size 1.27 1.27)) (justify right bottom))
   )
   (label "~{FAULT}" (at 203.2 78.74 0)

Commit message: Removed reset pin on backplane
The connection between the reset pin and the backplane has been removed
as it is not required. The reset pin on the backplane served no function
as it would be near impossible to use in practice and was likely to
cause issues surrounding pullup resistors if too many boards were added.
As such, the link between the backplane and the IC reset pins has been
removed, leaving only the reset button on the board.

Fixes #1

Signed-off-by: Matthew Nickson <mnickson@sidingsmedia.com>
Connections:
- net ~{RESET}: no longer J1.b10 (Pin_b10)
- no-connect marks 31 -> 32
Other:
- title: Speed controller -> Speed Control Node
Changed lines of the file:
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@@
   (paper "A4")
   (title_block
-    (title "Speed controller")
-    (date "2022-11-26")
-    (rev "0.3")
+    (title "Speed Control Node")
+    (date "2022-12-20")
+    (rev "0.4")
     (company "Sidings Media")
     (comment 1 "Licence: CERN-OHL-P-2.0 or any later version")
@@
   (no_connect (at 82.55 181.61))
   (no_connect (at 82.55 158.75))
+  (no_connect (at 49.53 48.26))
   (no_connect (at 49.53 38.1))
   (no_connect (at 49.53 35.56))
@@
     (stroke (width 0) (type default) (color 0 0 0 0))
   )
-  (wire (pts (xy 49.53 48.26) (xy 63.5 48.26))
-    (stroke (width 0) (type default) (color 0 0 0 0))
-  )
   (wire (pts (xy 22.86 105.41) (xy 22.86 107.95))
     (stroke (width 0) (type default) (color 0 0 0 0))
@@
     (effects (font (size 1.27 1.27)) (justify right bottom))
   )
-  (label "~{RESET}" (at 63.5 48.26 180)
-    (effects (font (size 1.27 1.27)) (justify right bottom))
-  )
