File: attiny84/motor_driver.kicad_sch (KiCad schematic)
At the start: 16 parts, among them J3 Screw_Terminal_01x03, J4 Screw_Terminal_01x03, J5 Screw_Terminal_01x03, J6 Screw_Terminal_01x03, Q3 BT138-800, U4 DRV8872DDA

Commit message: Assigned footprints to all components
Signed-off-by: Matthew Nickson <mnickson@sidingsmedia.com>
Parts:
- C6: footprint (none) -> Capacitor_SMD:C_1206_3216Metric_Pad1.33x1.80mm_HandSolder
- C7: footprint (none) -> Capacitor_SMD:CP_Elec_6.3x5.7
- C8: footprint Capacitor_THT:C_Disc_D4.7mm_W2.5mm_P5.00mm -> Capacitor_SMD:C_1206_3216Metric_Pad1.33x1.80mm_HandSolder
- D5: footprint (none) -> Diode_SMD:D_SOD-123F
- F1: footprint (none) -> Fuse:Fuseholder_Littelfuse_445_030_series_5x20mm
- J3, J4, J5, J6: footprint (none) -> TerminalBlock:TerminalBlock_bornier-3_P5.08mm
- R19: footprint (none) -> Resistor_SMD:R_1206_3216Metric_Pad1.30x1.75mm_HandSolder
Changed lines of the file:
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@@
       (effects (font (size 1.27 1.27)) (justify left))
     )
-    (property "Footprint" "Capacitor_THT:C_Disc_D4.7mm_W2.5mm_P5.00mm" (id 2) (at 169.8752 85.09 0)
+    (property "Footprint" "Capacitor_SMD:C_1206_3216Metric_Pad1.33x1.80mm_HandSolder" (id 2) (at 169.8752 85.09 0)
       (effects (font (size 1.27 1.27)) hide)
     )
@@
     (property "Reference" "F1" (id 0) (at 74.93 72.39 90))
     (property "Value" "5A" (id 1) (at 74.93 74.93 90))
-    (property "Footprint" "" (id 2) (at 74.93 80.518 90)
+    (property "Footprint" "Fuse:Fuseholder_Littelfuse_445_030_series_5x20mm" (id 2) (at 74.93 80.518 90)
       (effects (font (size 1.27 1.27)) hide)
     )
@@
       (effects (font (size 1.27 1.27)) (justify left))
     )
-    (property "Footprint" "" (id 2) (at 82.55 85.09 0)
+    (property "Footprint" "Diode_SMD:D_SOD-123F" (id 2) (at 82.55 85.09 0)
       (effects (font (size 1.27 1.27)) hide)
     )
@@
       (effects (font (size 1.27 1.27)) (justify left))
     )
-    (property "Footprint" "" (id 2) (at 80.772 97.79 90)
+    (property "Footprint" "Resistor_SMD:R_1206_3216Metric_Pad1.30x1.75mm_HandSolder" (id 2) (at 80.772 97.79 90)
       (effects (font (size 1.27 1.27)) hide)
     )
@@
       (effects (font (size 1.27 1.27)) (justify left))
     )
-    (property "Footprint" "" (id 2) (at 92.4052 101.6 0)
+    (property "Footprint" "Capacitor_SMD:C_1206_3216Metric_Pad1.33x1.80mm_HandSolder" (id 2) (at 92.4052 101.6 0)
       (effects (font (size 1.27 1.27)) hide)
     )
@@
       (effects (font (size 1.27 1.27)) (justify left))
     )
-    (property "Footprint" "" (id 2) (at 157.1752 85.09 0)
+    (property "Footprint" "Capacitor_SMD:CP_Elec_6.3x5.7" (id 2) (at 157.1752 85.09 0)
       (effects (font (size 1.27 1.27)) hide)
     )
@@
     (property "Reference" "J3" (id 0) (at 54.61 96.52 0))
     (property "Value" "Screw_Terminal_01x03" (id 1) (at 54.61 99.06 0))
-    (property "Footprint" "" (id 2) (at 54.61 105.41 0)
+    (property "Footprint" "TerminalBlock:TerminalBlock_bornier-3_P5.08mm" (id 2) (at 54.61 105.41 0)
       (effects (font (size 1.27 1.27)) hide)
     )
@@
       (effects (font (size 1.27 1.27)) (justify left))
     )
-    (property "Footprint" "" (id 2) (at 227.33 113.03 0)
+    (property "Footprint" "TerminalBlock:TerminalBlock_bornier-3_P5.08mm" (id 2) (at 227.33 113.03 0)
       (effects (font (size 1.27 1.27)) hide)
     )
@@
       (effects (font (size 1.27 1.27)) (justify left))
     )
-    (property "Footprint" "" (id 2) (at 55.88 78.74 0)
+    (property "Footprint" "TerminalBlock:TerminalBlock_bornier-3_P5.08mm" (id 2) (at 55.88 78.74 0)
       (effects (font (size 1.27 1.27)) hide)
     )
@@
       (effects (font (size 1.27 1.27)) (justify left))
     )
-    (property "Footprint" "" (id 2) (at 227.33 102.87 0)
-      (effects (font (size 1.27 1.27)) hide)
-    )
+    (property "Footprint" "TerminalBlock:TerminalBlock_bornier-3_P5.08mm" (id 2) (at 227.33 102.87 0)
+      (effects (font (size 1.27 1.27)) hide)
+    )

Commit message: Removed reset pin on backplane
The connection between the reset pin and the backplane has been removed
as it is not required. The reset pin on the backplane served no function
as it would be near impossible to use in practice and was likely to
cause issues surrounding pullup resistors if too many boards were added.
As such, the link between the backplane and the IC reset pins has been
removed, leaving only the reset button on the board.

Fixes #1

Signed-off-by: Matthew Nickson <mnickson@sidingsmedia.com>
Other:
- title: Speed controller -> Speed Control Node
Changed lines of the file:
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@@
   (paper "A4")
   (title_block
-    (title "Speed controller")
-    (date "2022-11-26")
-    (rev "0.3")
+    (title "Speed Control Node")
+    (date "2022-12-20")
+    (rev "0.4")
     (company "Sidings Media")
     (comment 1 "Licence: CERN-OHL-P-2.0 or any later version")
